File: K_Board.kicad_pcb (KiCad board)
At the start: 2 copper layers, 80 x 60 mm, 457 parts, among them J2 Conn_01x04, J3 Conns_I2C, J4 Conn_02x18_Counter_Clockwise, J5 USB pins, Q1 2N7002, Q2 AO3401A, Q3 2N7002, Q4 2N7002, SW10 Mechanical_Switch, SW11 Mechanical_Switch, SW12 Mechanical_Switch, SW13 K2-1187SQ-A4SW-06, SW14 Mechanical_Switch, SW15 Mechanical_Switch, SW16 Mechanical_Switch, SW17 Mechanical_Switch, SW18 Mechanical_Switch, SW2 Mechanical_Switch, SW20 Mechanical_Switch, SW21 Mechanical_Switch, SW22 Mechanical_Switch, SW23 Mechanical_Switch, SW25 Mechanical_Switch, SW26 Mechanical_Switch, SW27 Mechanical_Switch, SW28 Mechanical_Switch, SW3 Mechanical_Switch, SW30 Mechanical_Switch, SW31 Mechanical_Switch, SW32 Mechanical_Switch, SW33 Mechanical_Switch, SW35 Mechanical_Switch, SW36 Mechanical_Switch, SW37 Mechanical_Switch, SW38 Mechanical_Switch, SW39 Mechanical_Switch, SW4 Mechanical_Switch, SW41 Mechanical_Switch, SW42 Mechanical_Switch, SW43 Mechanical_Switch, SW44 Mechanical_Switch, SW46 Mechanical_Switch, SW47 Mechanical_Switch, SW48 Mechanical_Switch, SW49 Mechanical_Switch, SW5 Mechanical_Switch, SW51 Mechanical_Switch, SW52 Mechanical_Switch, SW53 Mechanical_Switch, SW54 Mechanical_Switch, SW56 Mechanical_Switch, SW57 Mechanical_Switch, SW58 Mechanical_Switch, SW59 Mechanical_Switch, SW6 Mechanical_Switch, SW60 Mechanical_Switch, SW62 Mechanical_Switch, SW63 Mechanical_Switch, SW64 Mechanical_Switch, SW65 Mechanical_Switch, SW66 Mechanical_Switch, SW68 Mechanical_Switch, SW69 Mechanical_Switch, SW7 Mechanical_Switch, SW72 Mechanical_Switch, SW73 Mechanical_Switch, SW74 Mechanical_Switch, SW75 Mechanical_Switch, SW76 Mechanical_Switch, SW77 Mechanical_Switch, SW78 Mechanical_Switch, SW79 Mechanical_Switch, SW8 Mechanical_Switch, SW80 Mechanical_Switch, SW81 Mechanical_Switch, SW82 Mechanical_Switch, SW9 Mechanical_Switch, U1 AT24C256C-SSHL-T, U2 STM32F411CEU6, U3 SGM2007-3.3XN5/TR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

Commit message: 02092022
Parts:
- added C102: 100n, Capacitor_SMD:C_0402_1005Metric, B.Cu at (447.8, 313.1)
- added C103: 100n, Capacitor_SMD:C_0402_1005Metric, B.Cu at (451.7, 317.1)
- added C104: 100n, Capacitor_SMD:C_0402_1005Metric, B.Cu at (458.7, 321.1)
- added C105: 100n, Capacitor_SMD:C_0402_1005Metric, B.Cu at (451.7, 315.1)
- added C106: 100n, Capacitor_SMD:C_0402_1005Metric, B.Cu at (442.1, 305.1)
- added C107: 100n, Capacitor_SMD:C_0402_1005Metric, B.Cu at (455.8, 320.2)
- added C108: 100n, Capacitor_SMD:C_0402_1005Metric, B.Cu at (442.1, 307.1)
- added C109: 100n, Capacitor_SMD:C_0402_1005Metric, B.Cu at (446.5, 308.1)
- added C110: 100n, Capacitor_SMD:C_0402_1005Metric, B.Cu at (453.5, 313.1)
- added C111: 100n, Capacitor_SMD:C_0402_1005Metric, B.Cu at (456.1, 318.2)
- added C112: 100n, Capacitor_SMD:C_0402_1005Metric, B.Cu at (450.6, 313.1)
- added C113: 100n, Capacitor_SMD:C_0402_1005Metric, B.Cu at (463.9, 327.0)
- added C114: 100n, Capacitor_SMD:C_0402_1005Metric, B.Cu at (458.7, 323.1)
- added C115: 100n, Capacitor_SMD:C_0402_1005Metric, F.Cu at (99.7, 86.1)
- added C116: 100n, Capacitor_SMD:C_0402_1005Metric, F.Cu at (107.9, 162.5)
- added D146: 1N4148W, Diode_SMD:D_SOD-123, F.Cu at (361.5, 72.2)
- added D147: 1N4148W, Diode_SMD:D_SOD-123, F.Cu at (337.6, 72.2)
- added D148: 1N4148W, Diode_SMD:D_SOD-123, F.Cu at (318.5, 72.2)
- added D149: 1N4148W, Diode_SMD:D_SOD-123, F.Cu at (299.6, 72.3)
- added D150: 1N4148W, Diode_SMD:D_SOD-123, F.Cu at (280.5, 72.3)
- added D151: 1N4148W, Diode_SMD:D_SOD-123, F.Cu at (256.6, 72.2)
- added D152: 1N4148W, Diode_SMD:D_SOD-123, F.Cu at (237.5, 72.2)
- added D153: 1N4148W, Diode_SMD:D_SOD-123, F.Cu at (218.5, 72.2)
- added D154: 1N4148W, Diode_SMD:D_SOD-123, F.Cu at (199.4, 72.2)
- added D155: 1N4148W, Diode_SMD:D_SOD-123, F.Cu at (175.5, 72.2)
- added D156: 1N4148W, Diode_SMD:D_SOD-123, F.Cu at (156.7, 72.2)
- added D157: 1N4148W, Diode_SMD:D_SOD-123, F.Cu at (137.4, 72.2)
- added D158: 1N4148W, Diode_SMD:D_SOD-123, F.Cu at (118.5, 72.2)
- added D159: 1N4148W, Diode_SMD:D_SOD-123, F.Cu at (331.9, 42.4)
- added D160: 1N4148W, Diode_SMD:D_SOD-123, F.Cu at (94.7, 72.2)
- added D161: 1N4148W, Diode_SMD:D_SOD-123, F.Cu at (65.9, 91.2)
- added D162: WS2812B-Mini, LED_SMD:LED_SK6812_PLCC4_5.0x5.0mm_P3.2mm, B.Cu at (465.5, 311.7)
- added D163: WS2812B-Mini, LED_SMD:LED_SK6812_PLCC4_5.0x5.0mm_P3.2mm, B.Cu at (472.5, 321.8)
- added D164: WS2812B-Mini, LED_SMD:LED_SK6812_PLCC4_5.0x5.0mm_P3.2mm, B.Cu at (479.5, 316.8)
- added D165: WS2812B-Mini, LED_SMD:LED_SK6812_PLCC4_5.0x5.0mm_P3.2mm, B.Cu at (479.5, 306.7)
- added D166: WS2812B-Mini, LED_SMD:LED_SK6812_PLCC4_5.0x5.0mm_P3.2mm, B.Cu at (472.5, 311.7)
- added D167: WS2812B-Mini, LED_SMD:LED_SK6812_PLCC4_5.0x5.0mm_P3.2mm, B.Cu at (458.4, 311.7)
- added D168: WS2812B-Mini, LED_SMD:LED_SK6812_PLCC4_5.0x5.0mm_P3.2mm, B.Cu at (451.4, 306.7)
- added D169: WS2812B-Mini, LED_SMD:LED_SK6812_PLCC4_5.0x5.0mm_P3.2mm, B.Cu at (479.5, 311.7)
- added D170: WS2812B-Mini, LED_SMD:LED_SK6812_PLCC4_5.0x5.0mm_P3.2mm, B.Cu at (465.5, 306.7)
- added D171: WS2812B-Mini, LED_SMD:LED_SK6812_PLCC4_5.0x5.0mm_P3.2mm, B.Cu at (458.4, 306.7)
- added D172: WS2812B-Mini, LED_SMD:LED_SK6812_PLCC4_5.0x5.0mm_P3.2mm, B.Cu at (479.5, 321.8)
- added D173: WS2812B-Mini, LED_SMD:LED_SK6812_PLCC4_5.0x5.0mm_P3.2mm, B.Cu at (472.5, 306.7)
- added D174: WS2812B-Mini, LED_SMD:LED_SK6812_PLCC4_5.0x5.0mm_P3.2mm, B.Cu at (472.5, 316.8)
- added D175: WS2812B-Mini, LED_SMD:LED_SK6812_PLCC4_5.0x5.0mm_P3.2mm, B.Cu at (99.7, 87.7)
- added D176: WS2812B-Mini, LED_SMD:LED_SK6812_PLCC4_5.0x5.0mm_P3.2mm, B.Cu at (107.8, 164.1)
- added R112: 5.1R, Resistor_SMD:R_0805_2012Metric, B.Cu at (459.7, 315.7)
- added R113: 5.1R, Resistor_SMD:R_0805_2012Metric, B.Cu at (445.7, 305.6)
- added R114: 5.1R, Resistor_SMD:R_0805_2012Metric, B.Cu at (476.4, 325.8)
- added R115: 5.1R, Resistor_SMD:R_0805_2012Metric, B.Cu at (448.3, 310.7)
- added R116: 5.1R, Resistor_SMD:R_0805_2012Metric, B.Cu at (466.8, 323.7)
- added R117: 5.1R, Resistor_SMD:R_0805_2012Metric, B.Cu at (459.7, 318.7)
- added R118: 5.1R, Resistor_SMD:R_0805_2012Metric, B.Cu at (472.0, 325.8)
- added R119: 5.1R, Resistor_SMD:R_0805_2012Metric, B.Cu at (462.4, 321.6)
- added R120: 5.1R, Resistor_SMD:R_0805_2012Metric, B.Cu at (455.3, 315.7)
- added R121: 5.1R, Resistor_SMD:R_0805_2012Metric, B.Cu at (480.8, 325.8)
- added R122: 5.1R, Resistor_SMD:R_0805_2012Metric, B.Cu at (467.6, 326.7)
- added R123: 5.1R, Resistor_SMD:R_0805_2012Metric, B.Cu at (466.8, 320.8)
- added R124: 5.1R, Resistor_SMD:R_0805_2012Metric, B.Cu at (452.7, 310.7)
- added R125: 5.1R, Resistor_SMD:R_0805_2012Metric, F.Cu at (99.7, 87.7)
- added R126: 5.1R, Resistor_SMD:R_0805_2012Metric, F.Cu at (107.9, 164.1)
- added SW1: EC11E1544407, Keebio-Parts:RotaryEncoder_Alps_EC11E-Switch_Vertical_H20mm, F.Cu at (60.6, 75.2)
- added SW19: Mechanical_Switch, acheron_MX_soldermask:MX100, F.Cu at (360.4, 78.7)
- added SW24: Mechanical_Switch, acheron_MX_soldermask:MX100, F.Cu at (336.6, 78.7)
- added SW29: Mechanical_Switch, acheron_MX_soldermask:MX100, F.Cu at (317.5, 78.7)
- added SW34: Mechanical_Switch, acheron_MX_soldermask:MX100, F.Cu at (298.5, 78.7)
- added SW40: Mechanical_Switch, acheron_MX_soldermask:MX100, F.Cu at (279.4, 78.7)
- added SW45: Mechanical_Switch, acheron_MX_soldermask:MX100, F.Cu at (255.6, 78.7)
- added SW50: Mechanical_Switch, acheron_MX_soldermask:MX100, F.Cu at (236.6, 78.7)
- added SW55: Mechanical_Switch, acheron_MX_soldermask:MX100, F.Cu at (217.5, 78.7)
- added SW61: Mechanical_Switch, acheron_MX_soldermask:MX100, F.Cu at (198.5, 78.7)
- added SW67: Mechanical_Switch, acheron_MX_soldermask:MX100, F.Cu at (174.6, 78.7)
- added SW70: Mechanical_Switch, acheron_MX_soldermask:MX100, F.Cu at (155.6, 78.7)
- added SW71: Mechanical_Switch, acheron_MX_soldermask:MX100, F.Cu at (136.6, 78.7)
- added SW83: Mechanical_Switch, acheron_MX_soldermask:MX100, F.Cu at (117.5, 78.7)
- added SW84: Mechanical_Switch, acheron_MX_soldermask:MX100, F.Cu at (127.0, 154.9)
- added SW85: Mechanical_Switch, acheron_MX_soldermask:MX100, F.Cu at (93.7, 78.7)
- added SW86: Mechanical_Switch, acheron_MX_soldermask:MX100, F.Cu at (60.4, 97.8)
- D1, D100, D101, D102, D103, D104, D105, D106, D107, D108, D109, D110, D111, D112, D113, D114, D115, D116, D117, D118, D119, D120, D121, D122, D123, D124, D125, D126, D127, D129, D13, D19, D24, D29, D34, D40, D45, D50, D55, D61, D67, D7, D70, D71, D83, D85, D86, D87, D88, D89, D90, D91, D92, D93, D94, D95, D96, D97, D98, D99: footprint LED_SMD:LED_SK6812MINI_PLCC4_3.5x3.5mm_P1.75mm -> LED_SMD:LED_SK6812_PLCC4_5.0x5.0mm_P3.2mm
- D128, D130, D131, D132, D133, D134, D135, D136, D137, D138, D139, D140, D141: footprint LED_SMD:LED_SK6812MINI_PLCC4_3.5x3.5mm_P1.75mm -> LED_SMD:LED_SK6812_PLCC4_5.0x5.0mm_P3.2mm; moved to B.Cu
- SW7: footprint acheron_MX_soldermask:MX225 -> acheron_MX_soldermask:MX_ISOEnter
- SW74: footprint acheron_MX_soldermask:MX150 -> acheron_MX_soldermask:MX100
- SW75: footprint acheron_MX_soldermask:MX175 -> acheron_MX_soldermask:MX100
- moved C88 685.4 mm to (60.1, 143.5), turned to 180 degrees
- moved C85 671.5 mm to (55.2, 83.6)
- moved R83 668.6 mm to (65.3, 85.2)
- moved R76 668.6 mm to (55.4, 65.0)
- moved R79 656.1 mm to (60.3, 125.9)
- moved R75 649.1 mm to (84.1, 188.0)
- moved C81 640.2 mm to (103.1, 186.3), turned to 180 degrees
- moved D80 634.5 mm to (92.7, 177.8), turned to 90 degrees
- moved C78 628.5 mm to (103.2, 105.2), turned to 180 degrees
- moved R74 626.4 mm to (84.1, 168.7)
- moved SW77 625.2 mm to (60.4, 116.8)
- moved D141 611.7 mm to (65.3, 85.2), turned to 180 degrees
- moved R81 610.0 mm to (65.0, 188.0)
- moved C86 609.6 mm to (60.3, 105.1), turned to 180 degrees
- moved D76 609.3 mm to (111.6, 177.8), turned to 90 degrees
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Connections:
- D125 pad 2: Net-(D125-Pad2) -> Net-(D136-Pad4)
- D129 pad 2: Net-(D129-Pad2) -> Net-(D130-Pad4)
- D129 pad 4: Net-(D125-Pad2) -> Net-(D121-Pad2)
- D130 pad 4: Net-(D121-Pad2) -> Net-(D130-Pad4)
- D132 pad 4: Net-(D126-Pad2) -> Net-(D132-Pad4)
- D134 pad 4: RGB_5V -> Net-(D134-Pad4)
- D136 pad 4: Net-(D129-Pad2) -> Net-(D136-Pad4)
- D74 pad 1: L3 -> L4
- SW74 pad 1: C14 -> C13
- SW77 pad 1: C15 -> C16
- SW78 pad 1: C15 -> C16
- U6 pad 4: L2 -> L1
- U6 pad 5: L3 -> L2
- U6 pad 6: L4 -> L3
- U6 pad 7: L5 -> L4
- U6 pad 8: L6 -> L5
- U6 pad 9: unconnected-(U6-Pad9) -> L6
Routing:
- net Net-(C84-Pad2): track 0.00 -> 5.34 mm, vias 0 -> 1
- net Net-(C80-Pad2): track 0.00 -> 4.99 mm, vias 0 -> 1
- net Net-(C116-Pad2): track 0.00 -> 4.97 mm, vias 0 -> 1
- net Net-(C83-Pad2): track 0.00 -> 4.89 mm, vias 0 -> 1
- net Net-(C82-Pad2): track 0.00 -> 4.88 mm, vias 0 -> 1
- net Net-(C81-Pad2): track 0.00 -> 4.83 mm, vias 0 -> 1
- net Net-(C78-Pad2): track 0.00 -> 4.83 mm, vias 0 -> 1
- net Net-(C86-Pad2): track 0.00 -> 4.77 mm, vias 0 -> 1
- net Net-(C87-Pad2): track 0.00 -> 4.75 mm, vias 0 -> 1
- net Net-(C89-Pad2): track 0.00 -> 4.73 mm, vias 0 -> 1
- net Net-(C90-Pad2): track 0.00 -> 3.29 mm, vias 0 -> 1
- net Net-(C115-Pad2): track 0.00 -> 3.05 mm, vias 0 -> 1
- net Net-(C91-Pad2): track 0.00 -> 3.05 mm, vias 0 -> 1
- net Net-(C85-Pad2): track 0.00 -> 3.05 mm, vias 0 -> 1
- net Net-(C88-Pad2): track 0.00 -> 2.96 mm, vias 0 -> 1
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Other:
- board outline removed
- board text added: "D129"
