File: K_Board.kicad_sch (KiCad schematic)
At the start: 459 parts, among them J1 TYPE-C-31-M-12, J2 Conn_01x04, J3 Conns_I2C, J4 Conn_02x18_Counter_Clockwise, J5 USB pins, Q1 2N7002, Q2 AO3401A, Q3 2N7002, Q4 2N7002, SW1 EC11E1544407, SW10 Mechanical_Switch, SW11 Mechanical_Switch, SW12 Mechanical_Switch, SW13 K2-1187SQ-A4SW-06, SW14 Mechanical_Switch, SW15 Mechanical_Switch, SW16 Mechanical_Switch, SW17 Mechanical_Switch, SW18 Mechanical_Switch, SW2 Mechanical_Switch, SW20 Mechanical_Switch, SW21 Mechanical_Switch, SW22 Mechanical_Switch, SW23 Mechanical_Switch, SW25 Mechanical_Switch, SW26 Mechanical_Switch, SW27 Mechanical_Switch, SW28 Mechanical_Switch, SW3 Mechanical_Switch, SW30 Mechanical_Switch, SW31 Mechanical_Switch, SW32 Mechanical_Switch, SW33 Mechanical_Switch, SW35 Mechanical_Switch, SW36 Mechanical_Switch, SW37 Mechanical_Switch, SW38 Mechanical_Switch, SW39 Mechanical_Switch, SW4 Mechanical_Switch, SW41 Mechanical_Switch, SW42 Mechanical_Switch, SW43 Mechanical_Switch, SW44 Mechanical_Switch, SW46 Mechanical_Switch, SW47 Mechanical_Switch, SW48 Mechanical_Switch, SW49 Mechanical_Switch, SW5 Mechanical_Switch, SW51 Mechanical_Switch, SW52 Mechanical_Switch, SW53 Mechanical_Switch, SW54 Mechanical_Switch, SW56 Mechanical_Switch, SW57 Mechanical_Switch, SW58 Mechanical_Switch, SW59 Mechanical_Switch, SW6 Mechanical_Switch, SW60 Mechanical_Switch, SW62 Mechanical_Switch, SW63 Mechanical_Switch, SW64 Mechanical_Switch, SW65 Mechanical_Switch, SW66 Mechanical_Switch, SW68 Mechanical_Switch, SW69 Mechanical_Switch, SW7 Mechanical_Switch, SW72 Mechanical_Switch, SW73 Mechanical_Switch, SW74 Mechanical_Switch, SW75 Mechanical_Switch, SW76 Mechanical_Switch, SW77 Mechanical_Switch, SW78 Mechanical_Switch, SW79 Mechanical_Switch, SW8 Mechanical_Switch, SW80 Mechanical_Switch, SW81 Mechanical_Switch, SW82 Mechanical_Switch, SW9 Mechanical_Switch, U1 AT24C256C-SSHL-T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

Commit message: 02092022
Parts:
- added C102, C103, C104, C105, C106, C107, C108, C109, C110, C111, C112, C113, C114, C115, C116: 100n, Capacitor_SMD:C_0402_1005Metric, symbol Device:C_Small
- added D146, D147, D148, D149, D150, D151, D152, D153, D154, D155, D156, D157, D158, D159, D160, D161: 1N4148W, Diode_SMD:D_SOD-123, symbol Diode:1N4148W
- added D162, D163, D164, D165, D166, D167, D168, D169, D170, D171, D172, D173, D174, D175, D176: WS2812B-Mini, LED_SMD:LED_SK6812MINI_PLCC4_3.5x3.5mm_P1.75mm, symbol acheron_Symbols:SK6812
- added R112, R113, R114, R115, R116, R117, R118, R119, R120, R121, R122, R123, R124, R125, R126: 5.1R, Resistor_SMD:R_0805_2012Metric, symbol Device:R_Small_US
- added SW19, SW24, SW29, SW34, SW40, SW45, SW50, SW55, SW61, SW67, SW70, SW71, SW83, SW84: Mechanical_Switch, acheron_MX_soldermask:MX100, symbol acheron_Symbols:Mechanical_Switch
- added SW85, SW86: Mechanical_Switch, acheron_MX_soldermask:MX200, symbol acheron_Symbols:Mechanical_Switch
- SW1: footprint (none) -> Keebio-Parts:RotaryEncoder_Alps_EC11E-Switch_Vertical_H20mm
- SW2: Keycode ESC -> "
- SW64: Keycode ? -> ^
- SW74: footprint acheron_MX_soldermask:MX150 -> acheron_MX_soldermask:MX100
Connections:
- net 5V: now also R112.2, R113.2, R114.2, R115.2, R116.2, R117.2, R118.2, R119.2, R120.2, R121.2, R122.2, R123.2, R124.2, R125.2, R126.2
- net C1: now also SW19.1
- net C10: now also SW67.1
- net C11: now also SW70.1
- net C12: now also SW71.1
- net C13: now also SW74.1, SW83.1, SW84.1
- net C14: now also SW85.1; no longer SW74.1
- net C15: no longer SW77.1, SW78.1
- net C16: now also SW77.1, SW78.1, SW86.1
- net C2: now also SW24.1
- net C3: now also SW29.1
- net C4: now also SW34.1
- net C5: now also SW40.1
- net C6: now also SW45.1
- net C7: now also SW50.1
- net C8: now also SW55.1
- net C9: now also SW61.1
- net GND: now also C102.1, C103.1, C104.1, C105.1, C106.1, C107.1, C108.1, C109.1, C110.1, C111.1, C112.1, C113.1, C114.1, C115.1, C116.1, D162.3 (VSS/GND), D163.3 (VSS/GND), D164.3 (VSS/GND), D165.3 (VSS/GND), D166.3 (VSS/GND), D167.3 (VSS/GND), D168.3 (VSS/GND), D169.3 (VSS/GND), D170.3 (VSS/GND), D171.3 (VSS/GND), D172.3 (VSS/GND), D173.3 (VSS/GND), D174.3 (VSS/GND), D175.3 (VSS/GND), D176.3 (VSS/GND)
- net L2: now also U6.5 (P1), D161.1 (K); no longer U6.4 (P0)
- net L3: now also U6.6 (P2); no longer D74.1 (K), U6.5 (P1)
- net L4: now also D74.1 (K), U6.7 (P3); no longer U6.6 (P2)
- net L5: now also U6.8 (P4), D159.1 (K); no longer U6.7 (P3)
- net L6: now also U6.9 (P5); no longer U6.8 (P4)
- net RGB_5V: now also D162.4 (DIN); no longer D134.4 (DIN)
- net at D136.4 (DIN): now also D125.2 (DOUT); no longer D129.2 (DOUT)
- net at D129.4 (DIN): now also D121.2 (DOUT); no longer D125.2 (DOUT)
- net at D126.2 (DOUT): now also D176.4 (DIN); no longer D132.4 (DIN)
- net at D130.4 (DIN): now also D129.2 (DOUT); no longer D121.2 (DOUT)
- new net: C115.2, D175.1 (VDD), R125.1
- new net: C110.2, D170.1 (VDD), R120.1
- new net: C104.2, D164.1 (VDD), R114.1
- new net: D159.2 (A), SW84.2
- new net: D150.2 (A), SW40.2
- new net: D149.2 (A), SW34.2
- new net: C109.2, D169.1 (VDD), R119.1
- new net: D152.2 (A), SW50.2
- new net: C106.2, D166.1 (VDD), R116.1
- new net: D166.2 (DOUT), D167.4 (DIN)
- new net: D165.2 (DOUT), D166.4 (DIN)
- new net: C112.2, D172.1 (VDD), R122.1
- new net: D148.2 (A), SW29.2
- new net: D172.2 (DOUT), D173.4 (DIN)
- new net: D171.2 (DOUT), D172.4 (DIN)
- new net: D161.2 (A), SW86.2
- new net: C108.2, D168.1 (VDD), R118.1
- new net: D151.2 (A), SW45.2
- new net: C102.2, D162.1 (VDD), R112.1
- new net: D155.2 (A), SW67.2
- new net: C105.2, D165.1 (VDD), R115.1
- new net: D134.4 (DIN), D175.2 (DOUT)
- new net: D164.2 (DOUT), D165.4 (DIN)
- new net: D174.2 (DOUT), D175.4 (DIN)
- new net: C107.2, D167.1 (VDD), R117.1
- new net: D167.2 (DOUT), D168.4 (DIN)
- new net: D154.2 (A), SW61.2
- new net: D147.2 (A), SW24.2
- new net: C114.2, D174.1 (VDD), R124.1
- new net: C116.2, D176.1 (VDD), R126.1
- new net: C113.2, D173.1 (VDD), R123.1
- new net: D173.2 (DOUT), D174.4 (DIN)
- new net: D160.2 (A), SW85.2
- new net: D168.2 (DOUT), D169.4 (DIN)
- new net: C111.2, D171.1 (VDD), R121.1
- new net: D158.2 (A), SW83.2
- new net: D156.2 (A), SW70.2
- new net: D163.2 (DOUT), D164.4 (DIN)
- new net: D146.2 (A), SW19.2
- new net: C103.2, D163.1 (VDD), R113.1
- new net: D169.2 (DOUT), D170.4 (DIN)
- new net: D162.2 (DOUT), D163.4 (DIN)
- new net: D157.2 (A), SW71.2
- new net: D153.2 (A), SW55.2
- new net: D170.2 (DOUT), D171.4 (DIN)
- new net: D132.4 (DIN), D176.2 (DOUT)
- new net L1: D146.1 (K), D147.1 (K), D148.1 (K), D149.1 (K), D150.1 (K), D151.1 (K), D152.1 (K), D153.1 (K), D154.1 (K), D155.1 (K), D156.1 (K), D157.1 (K), D158.1 (K), D160.1 (K), U6.4 (P0)
- no-connect marks 16 -> 15
Other:
- moved on the sheet: D77, D78, SW77, SW78, X2
